Commit message: Added Plotter Gcop urdf; Working gcop ctrl code with latest version of gcop, Added Airbot5 with the latest quadcopter example

File: gcop_ctrl/params/airbot4.urdf (robot description, URDF)
Before this commit: robot Airbot, 8 links, 7 joints
Links:
- link airbase: geometry visual box size=0.3 0.1 0.5

File: gcop_ctrl/params/airbot4.xacro (robot description, xacro)
@@ -20,6 +20,6 @@
 			<origin rpy="0 0 0" xyz="0.0 0.0 0.05"/>
       <geometry>
-				 <mesh filename="package://gcop_urdf/meshes/pelican1.dae" scale="0.025 0.025 0.025"/>
-        <!--box size="0.3 ${l1} 0.5"/-->
+				 <!--mesh filename="package://gcop_urdf/meshes/pelican1.dae" scale="0.025 0.025 0.025"/-->
+        <box size="0.3 ${l1} 0.5"/>
       </geometry>
       <material name="blue">
