Commit message: Added modifications to cost function for better convergence and modified the xacro files to match gcop convention with 2dof arm

File: gcop_ctrl/params/airbot5.urdf (robot description, URDF)
Before this commit: robot Airbotwith2dofarm, 5 links, 4 joints
Joints:
- joint airbasetolink1: axis 0 -1 0 -> 0 1 0; limit lower=-0.26179938765 upper=1.83259571355 effort=30 velocity=10.0 -> lower=1.30899693825 upper=2.87979326415 effort=30 velocity=10.0
- joint link1tolink2: axis 0 -1 0 -> 0 1 0; limit lower=-3.1415926518 upper=1.5707963259 effort=30 velocity=10.0 -> lower=-1.5707963259 upper=3.1415926518 effort=30 velocity=10.0; origin xyz=-0.025 0 -0.175 rpy=0 0 0 -> xyz=0.025 0 0.175 rpy=0 0 0
- joint link2tolink3: origin xyz=0 0 -0.42 rpy=0 0 0 -> xyz=0 0 0.42 rpy=0 0 0

File: gcop_ctrl/params/airbot5.xacro (robot description, xacro)
@@ -41,5 +41,5 @@
   <link name="link1">
     <visual>
-      <origin rpy="0 0 0" xyz="0.0 0.0 ${-l1/2}"/>
+      <origin rpy="0 0 0" xyz="0.0 0.0 ${l1/2}"/>
       <material name="blue">
         <color rgba="0 0 0.8 1"/>
@@ -50,5 +50,5 @@
     </visual>
     <inertial>
-      <origin rpy="0 0 0" xyz="0.0 0.0 0.0"/>
+      <origin rpy="0 0 0" xyz="0.0 0.0 0.0"/><!-- Since motors are heavy they constitute most weight-->
       <xacro:compute_inertia_cuboid mass="${m1}" x="0.05" y="0.05" z="0.05"/>
     </inertial>
@@ -56,5 +56,5 @@
   <link name="link2">
     <visual>
-      <origin rpy="0 0 0" xyz="0.0 0.0 ${-l2/2}"/>
+      <origin rpy="0 0 0" xyz="0.0 0.0 ${l2/2}"/>
       <geometry>
         <box size="0.02 0.02 ${l2}"/>
@@ -71,5 +71,5 @@
   <link name="link3">
     <visual>
-      <origin rpy="0 0 0" xyz="0.0 0.0 ${-l3/2}"/>
+      <origin rpy="0 0 0" xyz="0.0 0.0 ${l3/2}"/>
       <geometry>
         <box size="0.02 0.1 ${l3}"/>
@@ -80,5 +80,5 @@
     </visual>
     <inertial>
-      <origin rpy="0 0 0" xyz="0.0 0.0 ${-l3/2}"/>
+      <origin rpy="0 0 0" xyz="0.0 0.0 ${l3/2}"/>
       <xacro:compute_inertia_cuboid mass="${m3}" x="0.02" y="0.02" z="${l3}"/>
     </inertial>
@@ -94,18 +94,20 @@
     <child link="link1"/>
     <origin rpy="0 0 0" xyz="${x0} 0 ${-z0}"/>
-    <axis xyz="0 -1 0"/>
-    <limit effort="30" velocity="10.0" lower="${-15*degtorad}" upper="${105*degtorad}"/>
+    <axis xyz="0 1 0"/>
+    <!--limit effort="30" velocity="10.0" lower="-${360*degtorad}" upper="${360*degtorad}"/-->
+    <limit effort="30" velocity="10.0" lower="${75*degtorad}" upper="${165*degtorad}"/>
   </joint>
   <joint name="link1tolink2" type="revolute">
     <parent link="link1"/>
     <child link="link2"/>
-    <origin rpy="0 0 0" xyz="${-x1} 0 ${-l1}"/>
-    <axis xyz="0 -1 0"/>
-    <limit effort="30" velocity="10.0" lower="-${180*degtorad}" upper="${90*degtorad}"/>
+    <origin rpy="0 0 0" xyz="${x1} 0 ${l1}"/>
+    <axis xyz="0 1 0"/>
+    <!--limit effort="30" velocity="10.0" lower="-${360*degtorad}" upper="${360*degtorad}"/-->
+    <limit effort="30" velocity="10.0" lower="-${90*degtorad}" upper="${180*degtorad}"/>
   </joint>
   <joint name="link2tolink3" type="fixed">
     <parent link="link2"/>
     <child link="link3"/>
-    <origin rpy="0 0 0" xyz="0 0 ${-l2}"/>
+    <origin rpy="0 0 0" xyz="0 0 ${l2}"/>
   </joint>
 </robot>
