Commit message: Added new simple mesh with nurbs surface; and new carterrain with filled hole

File: gcop_ros_bullet/urdf/simple_mesh.urdf (robot description, URDF)
Before this commit: robot Mesh, 1 links, 0 joints
Links:
- link world: geometry visual mesh filename=package://gcop_ros_bullet/urdf/meshes/simple_mesh2.dae
