Commit message: Added support for separating base frame from base inertial frame

File: gcop_urdf/urdf/airbot_cyton.urdf (robot description, URDF)
Before this commit: robot airbot_cyton_gamma_1500, 11 links, 10 joints
Links:
- added link gripper_finger1, mass 0.05; collision box size=0.015 0.0229 0.0475; visual mesh filename=package://cyton_gamma_1500_description/meshes/gripper_finge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
- added link gripper_finger2, mass 0.05; collision box size=0.015 0.0229 0.0475; visual mesh filename=package://cyton_gamma_1500_description/meshes/gripper_finge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
- added link target, mass 1e-5; visual mesh filename=package://gcop_urdf/meshes/cordless_drill/cordless_drill.dae scale=1 1 1
- link airbase: geometry visual mesh filename=package://gcop_urdf/meshes/dji-s1000.dae scale=1 1 1
Joints:
- added joint endeffector_target_joint: type fixed, parent virtual_endeffector, child target, origin xyz=0 -0.22 0.06 rpy=1.57079632679 0 3.14159265359
- added joint gripper_joint: type fixed, parent wrist_roll, child gripper_finger1, origin xyz=-0.02 0.00485 0.077225 rpy=0.0 0 0
- added joint gripper_joint2: type fixed, parent wrist_roll, child gripper_finger2, origin xyz=0.02 0.00485 0.077225 rpy=0 0 0
- joint base_cyton_joint: origin xyz=0.0732 0.0 -0.1 rpy=3.14159265359 0 1.57079632679 -> xyz=0.076 0.0 -0.12 rpy=3.14159265359 0 1.57079632679

File: gcop_urdf/urdf/airbot_cyton.xacro (robot description, xacro)
@@ -4,6 +4,7 @@
   <xacro:include filename="$(find cyton_gamma_1500_description)/cyton_gamma_1500_macros.urdf.xacro"/>
   <xacro:property name="mass_airbot" value="4.2"/>
-  <xacro:property name="base_offset_x" value="0.0732"/>
-  <xacro:property name="base_offset_z" value="-0.1"/>
+  <xacro:property name="base_offset_x" value="0.076"/>
+  <!--<xacro:property name="base_offset_x" value="0.0"/>-->
+  <xacro:property name="base_offset_z" value="-0.12"/>
   <xacro:macro name="cylinder_inertia" params="mass d h">
         <inertia
@@ -30,10 +31,7 @@
       <origin rpy="0 0 0" xyz="0.0 0.0 0.0"/>
       <geometry>
-        <mesh filename="package://gcop_urdf/meshes/quadrotor_base.dae" scale="3 3 1"/>
+        <mesh filename="package://gcop_urdf/meshes/dji-s1000.dae" scale="1 1 1"/>
         <!--box size="0.44 0.44 0.1632"/-->
       </geometry>
-      <material name="red">
-        <color rgba="0.8 0 0 1"/>
-      </material>
     </visual>
     <inertial>
@@ -54,3 +52,22 @@
   </joint>
   <xacro:cyton_gamma_1500 prefix="" virtual_ee="true"/>
+  <!-- Add an electric drill visual at the end of gripper-->
+  <link name="target">
+    <visual>
+      <origin rpy="0 0 0" xyz="0.0 0.0 0.0"/>
+      <geometry>
+        <mesh filename="package://gcop_urdf/meshes/cordless_drill/cordless_drill.dae" scale="1 1 1"/>
+      </geometry>
+    </visual>
+    <inertial>
+      <origin rpy="0 0 0" xyz="0 0 0"/>
+      <mass value="1e-5"/>
+      <inertia ixx="6.66666666667e-12" ixy="0.0" ixz="0.0" iyy="6.66666666667e-12" iyz="0.0" izz="6.66666666667e-12"/>
+    </inertial>
+  </link>
+  <joint name="endeffector_target_joint" type="fixed">
+      <parent link="virtual_endeffector" />
+      <child link="target" />
+      <origin xyz="0 -0.22 0.06" rpy="${pi/2} 0 ${pi}" />
+  </joint>
 </robot>
